File: hardware/tf2/tiny2313_ft232.kicad_pcb (KiCad board)
At the start: 2 copper layers, 63.5 x 48.3 mm, 35 parts

Commit message: tf2 bugfix
Connections:
- led_portD2 pad 1: Net-(led_portD2-Pad1) -> GND
- led_portD3 pad 1: Net-(led_portD2-Pad1) -> GND
- led_portD4 pad 1: Net-(led_portD2-Pad1) -> GND
- led_portD5 pad 1: Net-(led_portD2-Pad1) -> GND
- led_portD6 pad 1: Net-(led_portD2-Pad1) -> GND
Changed lines of the file:
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@@
-(kicad_pcb (version 20171130) (host pcbnew 5.0.0-rc2-dev-unknown-2da7199~62~ubuntu17.10.1)
+(kicad_pcb (version 20171130) (host pcbnew 5.0.0-rc2-dev-unknown-f1cf95b~62~ubuntu17.10.1)
   (general
     (thickness 1.6)
@@
     (zones 0)
     (modules 35)
-    (nets 57)
+    (nets 56)
   )
   (page A4)
@@
   (net 54 /PA1)
   (net 55 /PA0)
-  (net 56 "Net-(led_portD2-Pad1)")
   (net_class Default "This is the default net class."
     (clearance 0.2)
@@
     (add_net "Net-(ledR_portD5-Pad1)")
     (add_net "Net-(ledR_portD6-Pad1)")
-    (add_net "Net-(led_portD2-Pad1)")
   )
   (module Housings_DIP:DIP-28_W15.24mm_Socket (layer F.Cu)
@@
     (fp_line (start 4.5 -3.25) (end -1.95 -3.25) (layer F.CrtYd) (width 0.05))
     (pad 1 thru_hole rect (at 0 0 90) (size 1.8 1.8) (drill 0.9) (layers *.Cu *.Mask)
-      (net 56 "Net-(led_portD2-Pad1)"))
+      (net 1 GND))
     (pad 2 thru_hole circle (at 2.54 0 90) (size 1.8 1.8) (drill 0.9) (layers *.Cu *.Mask)
       (net 19 "Net-(ledR_portD4-Pad1)"))
@@
     (fp_line (start 4.5 -3.25) (end -1.95 -3.25) (layer F.CrtYd) (width 0.05))
     (pad 1 thru_hole rect (at 0 0 90) (size 1.8 1.8) (drill 0.9) (layers *.Cu *.Mask)
-      (net 56 "Net-(led_portD2-Pad1)"))
+      (net 1 GND))
     (pad 2 thru_hole circle (at 2.54 0 90) (size 1.8 1.8) (drill 0.9) (layers *.Cu *.Mask)
       (net 17 "Net-(ledR_portD2-Pad1)"))
@@
       (net 18 "Net-(ledR_portD3-Pad1)"))
     (pad 1 thru_hole rect (at 0 0 90) (size 1.8 1.8) (drill 0.9) (layers *.Cu *.Mask)
-      (net 56 "Net-(led_portD2-Pad1)"))
+      (net 1 GND))
     (model LEDs.3dshapes/LED_D5.0mm.wrl
       (at (xyz 0 0 0))
@@
       (net 20 "Net-(ledR_portD5-Pad1)"))
     (pad 1 thru_hole rect (at 0 0 90) (size 1.8 1.8) (drill 0.9) (layers *.Cu *.Mask)
-      (net 56 "Net-(led_portD2-Pad1)"))
+      (net 1 GND))
     (model LEDs.3dshapes/LED_D5.0mm.wrl
       (at (xyz 0 0 0))
@@
     (fp_line (start 4.5 -3.25) (end -1.95 -3.25) (layer F.CrtYd) (width 0.05))
     (pad 1 thru_hole rect (at 0 0 90) (size 1.8 1.8) (drill 0.9) (layers *.Cu *.Mask)
-      (net 56 "Net-(led_portD2-Pad1)"))
+      (net 1 GND))
     (pad 2 thru_hole circle (at 2.54 0 90) (size 1.8 1.8) (drill 0.9) (layers *.Cu *.Mask)
       (net 21 "Net-(ledR_portD6-Pad1)"))

Commit message: add host library template driver and python example
Connections:
- net /PB5 renamed /PB5-MOSI
- net /PB6 renamed /PB6-MISO
- net /PB7 renamed /PB7-SCK
